File: KDT_Hierarchical_KiBot.kicad_sch (KiCad schematic)
At the start: 0 parts

Commit message: Updated template
Other:
- note added: "NOTE STYLING CONVENTION"
- note added: "STATUS CONVENTION"
- note added: "Status: ${VARIANT}"
- note removed: "CHECKED - There shouldn't be any mistakes. Contact the engineer if you find any."
- note removed: "Comment"
- note removed: "DESIGN CONSIDERATIONS"
- note removed: "DRAFT - Very early stage of schematic, ignore details."
- note removed: "NOTES"
- note removed: "Not fitted components are marked as"
- note removed: "PRELIMINARY - Close to final schematic."
- note removed: "RELEASED - A board with this schematic has been sent to production."
- note removed: "Variant: ${VARIANT}"
